File: main-board.kicad_sch (KiCad schematic)
At the start: 10 parts, among them IC1 FS312F-G, J1 BAT_NEG, J2 POS_OUT, J3 BAT_POS, J4 NEG_OUT, Q1 FS8205A

Commit message: minor
Other:
- moved on the sheet: J1, J3
Changed lines of the file:
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@@
     )
   )
-  (global_label "BAT_NEG" (shape input) (at 232.41 85.09 180) (fields_autoplaced)
+  (global_label "BAT_NEG" (shape input) (at 123.19 121.92 180) (fields_autoplaced)
     (effects (font (size 1.27 1.27)) (justify right))
-    (property "Intersheet References" "${INTERSHEET_REFS}" (id 0) (at 222.0425 85.1694 0)
+    (property "Intersheet References" "${INTERSHEET_REFS}" (id 0) (at 112.8225 121.9994 0)
       (effects (font (size 1.27 1.27)) (justify right) hide)
     )
@@
     )
   )
-  (global_label "BAT_POS" (shape input) (at 232.41 90.805 180) (fields_autoplaced)
+  (global_label "BAT_POS" (shape input) (at 123.19 127.635 180) (fields_autoplaced)
     (effects (font (size 1.27 1.27)) (justify right))
-    (property "Intersheet References" "${INTERSHEET_REFS}" (id 0) (at 221.982 90.7256 0)
+    (property "Intersheet References" "${INTERSHEET_REFS}" (id 0) (at 112.762 127.5556 0)
       (effects (font (size 1.27 1.27)) (justify right) hide)
     )
@@
     (pin "2")
   )
-  (symbol (lib_id "Connector:Conn_01x01_Female") (at 237.49 85.09 0) (unit 1)
+  (symbol (lib_id "Connector:Conn_01x01_Female") (at 128.27 121.92 0) (unit 1)
     (in_bom yes) (on_board yes)
-    (property "Reference" "J1" (id 0) (at 240.03 84.455 0)
-      (effects (font (size 1.27 1.27)) (justify left))
-    )
-    (property "Value" "BAT_NEG" (id 1) (at 238.125 86.36 0)
-      (effects (font (size 1.27 1.27)) (justify left))
-    )
-    (property "Footprint" "Connector_Wire:SolderWirePad_1x01_SMD_1x2mm" (id 2) (at 237.49 85.09 0)
-      (effects (font (size 1.27 1.27)) hide)
-    )
-    (property "Datasheet" "~" (id 3) (at 237.49 85.09 0)
-      (effects (font (size 1.27 1.27)) hide)
-    )
-    (pin "1")
-  )
-  (symbol (lib_id "Connector:Conn_01x01_Female") (at 237.49 90.805 0) (unit 1)
+    (property "Reference" "J1" (id 0) (at 130.81 121.285 0)
+      (effects (font (size 1.27 1.27)) (justify left))
+    )
+    (property "Value" "BAT_NEG" (id 1) (at 128.905 123.19 0)
+      (effects (font (size 1.27 1.27)) (justify left))
+    )
+    (property "Footprint" "Connector_Wire:SolderWirePad_1x01_SMD_1x2mm" (id 2) (at 128.27 121.92 0)
+      (effects (font (size 1.27 1.27)) hide)
+    )
+    (property "Datasheet" "~" (id 3) (at 128.27 121.92 0)
+      (effects (font (size 1.27 1.27)) hide)
+    )
+    (pin "1")
+  )
+  (symbol (lib_id "Connector:Conn_01x01_Female") (at 128.27 127.635 0) (unit 1)
     (in_bom yes) (on_board yes)
-    (property "Reference" "J3" (id 0) (at 240.665 90.17 0)
-      (effects (font (size 1.27 1.27)) (justify left))
-    )
-    (property "Value" "BAT_POS" (id 1) (at 238.2012 92.6716 0)
-      (effects (font (size 1.27 1.27)) (justify left))
-    )
-    (property "Footprint" "Connector_Wire:SolderWirePad_1x01_SMD_1x2mm" (id 2) (at 237.49 90.805 0)
-      (effects (font (size 1.27 1.27)) hide)
-    )
-    (property "Datasheet" "~" (id 3) (at 237.49 90.805 0)
-      (effects (font (size 1.27 1.27)) hide)
-    )
+    (property "Reference" "J3" (id 0) (at 131.445 127 0)
+      (effects (font (size 1.27 1.27)) (justify left))
+    )
+    (property "Value" "BAT_POS" (id 1) (at 128.9812 129.5016 0)
+      (effects (font (size 1.27 1.27)) (justify left))
+    )
+    (property "Footprint" "Connector_Wire:SolderWirePad_1x01_SMD_1x2mm" (id 2) (at 128.27 127.635 0)
+      (effects (font (size 1.27 1.27)) hide)
+    )
+    (property "Datasheet" "~" (id 3) (at 128.27 127.635 0)
+      (effects (font (size 1.27 1.27)) hide)
+    )
